Commit message: update readme

File: car_model/spawn_car/model/mevi/urdf/mevi_description.urdf.xacro (robot description, xacro)
@@ -21,10 +21,10 @@
     <xacro:Rear_Right_Wheel/>
     <xacro:Rear_Left_Wheel/>
-    <!-- <xacro:rgb_camera frlr_prefix="front" lrc_prefix="center">
+    <xacro:rgb_camera frlr_prefix="front" lrc_prefix="center">
       <origin xyz="-0.04 0 1" rpy="0 0.087 0"/>
     </xacro:rgb_camera>
     <xacro:VLP-16 parent="chassis" name="velodyne" topic="/velodyne_points" organize_cloud="${organize_cloud}" hz="10" samples="440" gpu="${gpu}">
       <origin xyz="0 0 0.4" rpy="0 0 0" />
-    </xacro:VLP-16> -->
+    </xacro:VLP-16>
       <gazebo>
         <plugin name="p3d" filename="libgazebo_ros_p3d.so">

File: car_model/spawn_car/model/mevi/urdf/sensors/camera.urdf.xacro (robot description, xacro)
@@ -64,5 +64,5 @@
                     <alwaysOn>true</alwaysOn>
                     <updateRate>0.0</updateRate>
-                    <cameraName>sd_twizy/${frlr_prefix}_${lrc_prefix}_camera</cameraName>
+                    <cameraName>mevi/${frlr_prefix}_${lrc_prefix}_camera</cameraName>
                     <imageTopicName>image_raw</imageTopicName>
                     <cameraInfoTopicName>camera_info</cameraInfoTopicName>

File: car_model/spawn_car/model/mevi/urdf/sensors/vlp-16.urdf.xacro (robot description, xacro)
@@ -18,10 +18,10 @@
         <visual>
             <geometry>
-            <mesh filename="package://spawn_car/model/meshes/VLP16_base_1.dae" />
+            <mesh filename="package://spawn_car/model/mevi/meshes/VLP16_base_1.dae" />
             </geometry>
         </visual>
         <visual>
             <geometry>
-            <mesh filename="package://spawn_car/model/meshes/VLP16_base_2.dae" />
+            <mesh filename="package://spawn_car/model/mevi/meshes/VLP16_base_2.dae" />
             </geometry>
         </visual>
@@ -47,5 +47,5 @@
             <origin xyz="0 0 -0.0377" />
             <geometry>
-            <mesh filename="package://spawn_car/model/meshes/VLP16_scan.dae" />
+            <mesh filename="package://spawn_car/model/mevi/meshes/VLP16_scan.dae" />
             </geometry>
         </visual>

Commit message: fixes simulation

File: car_model/spawn_car/model/mevi/urdf/mevi_description.urdf.xacro (robot description, xacro)
@@ -21,10 +21,10 @@
     <xacro:Rear_Right_Wheel/>
     <xacro:Rear_Left_Wheel/>
-    <xacro:rgb_camera frlr_prefix="front" lrc_prefix="center">
+    <!-- <xacro:rgb_camera frlr_prefix="front" lrc_prefix="center">
       <origin xyz="-0.04 0 1" rpy="0 0.087 0"/>
     </xacro:rgb_camera>
     <xacro:VLP-16 parent="chassis" name="velodyne" topic="/velodyne_points" organize_cloud="${organize_cloud}" hz="10" samples="440" gpu="${gpu}">
       <origin xyz="0 0 0.4" rpy="0 0 0" />
-    </xacro:VLP-16>
+    </xacro:VLP-16> -->
       <gazebo>
         <plugin name="p3d" filename="libgazebo_ros_p3d.so">

File: car_model/spawn_car/model/mevi/urdf/wheels/mevi_suspension.urdf.xacro (robot description, xacro)
@@ -54,5 +54,5 @@
             <parent link="chassis"/>
             <child link="fl_axle"/>
-            <origin rpy="${degree_90} 0 0" xyz="${-wheel_base/2} ${-front_track/2} 0"/>
+            <origin rpy="${degree_90} 0 0" xyz="${wheel_base/2} ${-front_track/2} 0"/>
             <axis xyz="0 1 0"/>
             <limit lower="-0.785398" upper="0.785398" effort="500000" velocity="250"/>
@@ -71,5 +71,5 @@
             <parent link="chassis"/>
             <child link="fr_axle"/>
-            <origin rpy="${degree_90} 0 0" xyz="${-wheel_base/2} ${front_track/2} 0"/>
+            <origin rpy="${degree_90} 0 0" xyz="${wheel_base/2} ${front_track/2} 0"/>
             <axis xyz="0 1 0"/>
             <limit lower="-0.785398" upper="0.785398" effort="500000" velocity="250"/>
@@ -88,5 +88,5 @@
             <parent link="chassis"/>
             <child link="rear_left_wheel"/>
-            <origin rpy="${degree_90} 0 0" xyz="${wheel_base/2} ${-front_track/2} 0"/>
+            <origin rpy="${degree_90} 0 0" xyz="${-wheel_base/2} ${-front_track/2} 0"/>
             <axis xyz="0 0 -1"/>
             <limit effort="1000" velocity="1000"/>
@@ -98,5 +98,5 @@
             <parent link="chassis"/>
             <child link="rear_right_wheel"/>
-            <origin rpy="${degree_90} 0 0" xyz="${wheel_base/2} ${front_track/2} 0"/>
+            <origin rpy="${degree_90} 0 0" xyz="${-wheel_base/2} ${front_track/2} 0"/>
             <axis xyz="0 0 -1"/>
             <limit effort="1000" velocity="1000"/>
