Commit message: adding mesh from twizy

File: spawn_car/model/mevi/urdf/bases/mevi_body.urdf.xacro (robot description, xacro)
@@ -27,5 +27,5 @@
         </joint>
         <link name="chassis">
-            <visual>
+            <!-- <visual>
                 <origin xyz="0 0 0" rpy="0 0 0"/>
                 <geometry>
@@ -33,9 +33,15 @@
                 </geometry>
                 <material name="chassis_mat"/>
-            </visual>
+            </visual> -->
+            <visual>
+                <origin xyz="0.015 0.0 0.015" rpy="0 0 1.57079632679"/>
+                <geometry>
+                  <mesh filename="file://$(find spawn_car)/model/mevi/meshes/SDTwizy.stl" scale="0.008 0.0055 0.0062"/>
+                </geometry>
+              </visual>
             <collision>
-                <origin xyz="0 0 0" rpy="0 0 0"/>
+                <origin xyz="0.015 0.0 0.015" rpy="0 0 1.57079632679"/>
                 <geometry>
-                    <box size="${chassis_length} ${chassis_width} ${chassis_thickness}"/>
+                  <mesh filename="file://$(find spawn_car)/model/mevi/meshes/SDTwizy_collision.stl" scale="0.008 0.0055 0.0062"/>
                 </geometry>
             </collision>

File: spawn_car/model/mevi/urdf/vehicle_properties.urdf.xacro (robot description, xacro)
@@ -33,4 +33,12 @@
     -->
     <xacro:property name="wheel_cylindrical_transform" value="1.570795" />
+    <xacro:property name="front_wheel_radius" value="0.172"/>
+    <xacro:property name="front_wheel_width" value="0.125"/>
+    <xacro:property name="front_wheel_mass" value="10.0"/>
+    <xacro:property name="rear_wheel_radius" value="0.172"/>
+    <xacro:property name="rear_wheel_width" value="0.125"/>
+    <xacro:property name="rear_wheel_mass" value="10.0"/>
+    <xacro:property name="front_track" value="0.830" />
+    <xacro:property name="rear_track" value="0.750" />
     <!-- mass -->
     <!-- let assume the mass of box same as half aluminium at it size-->

File: spawn_car/model/mevi/urdf/wheels/mevi_suspension.urdf.xacro (robot description, xacro)
@@ -10,12 +10,4 @@
     <xacro:include filename="$(find spawn_car)/model/mevi/urdf/wheels/suspension.gazebo.xacro"/>
     <xacro:include filename="$(find spawn_car)/model/mevi/urdf/vehicle_properties.urdf.xacro"/>
-    <xacro:property name="front_wheel_radius" value="0.185"/>
-    <xacro:property name="front_wheel_width" value="0.125"/>
-    <xacro:property name="front_wheel_mass" value="10.0"/>
-    <xacro:property name="rear_wheel_radius" value="0.185"/>
-    <xacro:property name="rear_wheel_width" value="0.125"/>
-    <xacro:property name="rear_wheel_mass" value="10.0"/>
-    <xacro:property name="front_track" value="0.830" />
-    <xacro:property name="rear_track" value="0.750" />
     <xacro:property name="Iz_rear_wheel" value="${0.5*rear_wheel_mass*rear_wheel_radius*rear_wheel_radius}"/>
     <xacro:property name="I_rear_wheel" value="${1/12*rear_wheel_mass*(3*rear_wheel_radius*rear_wheel_radius + rear_wheel_width*rear_wheel_width)}"/>
