Commit message: formula simulation worked

File: spawn_car/model/formula/urdf/bases/formula_body.gazebo.xacro (robot description, xacro)
@@ -6,6 +6,9 @@
 <robot xmlns:xacro="http://www.ros.org/wiki/xacro" name="formula">
     <gazebo reference="chassis">
-      <material name="sf24_livery" >
+      <!-- <material name="sf24_livery" >
         <color rgba="0.91 0.03 0.02 1.0" />
+      </material> -->
+      <material>
+        Gazebo/Red
       </material>
     </gazebo>

File: spawn_car/model/formula/urdf/bases/formula_body.urdf.xacro (robot description, xacro)
@@ -10,4 +10,7 @@
         <color rgba="0.2 0.2 0.2 1"/>
         <!-- grey -->
+    </material>
+    <material name="sf24_livery" >
+        <color rgba="0.91 0.03 0.02 1.0" />
     </material>
     <xacro:macro name="formula_base" params="name">
@@ -39,4 +42,8 @@
                   <mesh filename="file://$(find spawn_car)/model/formula/meshes/F1_2023_halo_livery.stl" scale="0.03 0.03 0.03"/>
                 </geometry>
+                <!-- <material name="sf24_livery"/> -->
+                <material name="sf24_livery" >
+                    <color rgba="0.91 0.03 0.02 1.0" />
+                </material>
             </visual>
             <collision>
@@ -45,4 +52,8 @@
                     <box size="${car_length} ${car_width} ${car_height - 0.6} "/>
                 </geometry>
+                <!-- <material name="sf24_livery" /> -->
+                <material name="sf24_livery" >
+                    <color rgba="0.91 0.03 0.02 1.0" />
+                </material>
             </collision>
             <xacro:inertia_of_body/>

File: spawn_car/model/formula/urdf/formula_description.urdf.xacro (robot description, xacro)
@@ -21,10 +21,10 @@
     <xacro:Rear_Right_Wheel/>
     <xacro:Rear_Left_Wheel/>
-    <xacro:rgb_camera frlr_prefix="front" lrc_prefix="center">
+    <!-- <xacro:rgb_camera frlr_prefix="front" lrc_prefix="center">
       <origin xyz="-0.04 0 1" rpy="0 0.087 0"/>
-    </xacro:rgb_camera>
-    <xacro:VLP-16 parent="chassis" name="velodyne" topic="/velodyne_points" organize_cloud="${organize_cloud}" hz="10" samples="440" gpu="${gpu}">
+    </xacro:rgb_camera> -->
+    <!-- <xacro:VLP-16 parent="chassis" name="velodyne" topic="/velodyne_points" organize_cloud="${organize_cloud}" hz="10" samples="440" gpu="${gpu}">
       <origin xyz="0 0 ${car_height - 0.23}" rpy="0 0 0" />
-    </xacro:VLP-16>
+    </xacro:VLP-16> -->
       <gazebo>
         <plugin name="p3d" filename="libgazebo_ros_p3d.so">

File: spawn_car/model/formula/urdf/sensors/camera.urdf.xacro (robot description, xacro)
@@ -4,4 +4,5 @@
     <joint name="${frlr_prefix}_${lrc_prefix}_camera_joint" type="fixed">
       <axis xyz="0 1 0" />
+      <origin xyz="0 0 ${car_height}" rpy="0 0 0"/>
       <xacro:insert_block name="origin"/>
       <!-- parent link dari camera adalah chassis -->

File: spawn_car/model/formula/urdf/wheels/formula_suspension.urdf.xacro (robot description, xacro)
@@ -143,4 +143,5 @@
                 <cylinder length="${front_tyre_width}" radius="${front_tyre_radius}"/>
             </geometry>
+            <material name="pirelli"/>
         </collision>
         <xacro:inertia_of_front_wheel/>
@@ -159,4 +160,5 @@
                 <cylinder length="${front_tyre_width}" radius="${front_tyre_radius}"/>
             </geometry>
+            <material name="pirelli"/>
         </collision>
         <xacro:inertia_of_front_wheel/>
@@ -175,4 +177,5 @@
                 <cylinder length="${rear_tyre_width}" radius="${rear_tyre_radius}"/>
             </geometry>
+            <material name="pirelli"/>
         </collision>
         <xacro:inertia_of_rear_wheel/>
@@ -191,4 +194,5 @@
                 <cylinder length="${rear_tyre_width}" radius="${rear_tyre_radius}"/>
             </geometry>
+            <material name="pirelli"/>
         </collision>
         <xacro:inertia_of_rear_wheel/>

File: spawn_car/model/formula/urdf/wheels/suspension.gazebo.xacro (robot description, xacro)
@@ -12,6 +12,9 @@
         <minDepth>0.005</minDepth>
         <kp>1e8</kp>
-        <material name="pirelli" >
+        <!-- <material name="pirelli" >
             <color rgba="0.35 0.35 0.35 1.0" />
+        </material> -->
+        <material>
+            Gazebo/Grey
         </material>
     </gazebo>
@@ -21,6 +24,9 @@
         <minDepth>0.005</minDepth>
         <kp>1e8</kp>
-        <material name="pirelli" >
+        <!-- <material name="pirelli" >
             <color rgba="0.35 0.35 0.35 1.0" />
+        </material> -->
+        <material>
+            Gazebo/Grey
         </material>
     </gazebo>
@@ -30,6 +36,9 @@
         <minDepth>0.005</minDepth>
         <kp>1e8</kp>
-        <material name="pirelli" >
+        <!-- <material name="pirelli" >
             <color rgba="0.35 0.35 0.35 1.0" />
+        </material> -->
+        <material>
+            Gazebo/Grey
         </material>
     </gazebo>
@@ -39,6 +48,9 @@
         <minDepth>0.005</minDepth>
         <kp>1e8</kp>
-        <material name="pirelli" >
+        <!-- <material name="pirelli" >
             <color rgba="0.35 0.35 0.35 1.0" />
+        </material> -->
+        <material>
+            Gazebo/Grey
         </material>
     </gazebo>
