Commit message: solving acckermann formula

File: spawn_car/model/formula/urdf/wheels/suspension.gazebo.xacro (robot description, xacro)
@@ -16,5 +16,5 @@
         </material> -->
         <material>
-            Gazebo/Grey
+            Gazebo/Black
         </material>
     </gazebo>
@@ -28,5 +28,5 @@
         </material> -->
         <material>
-            Gazebo/Grey
+            Gazebo/Black
         </material>
     </gazebo>
@@ -40,5 +40,5 @@
         </material> -->
         <material>
-            Gazebo/Grey
+            Gazebo/Black
         </material>
     </gazebo>
@@ -52,5 +52,5 @@
         </material> -->
         <material>
-            Gazebo/Grey
+            Gazebo/Black
         </material>
     </gazebo>

File: spawn_car/model/urban/urdf/urban_description.urdf.xacro (robot description, xacro)
@@ -21,10 +21,10 @@
     <xacro:Rear_Right_Wheel/>
     <xacro:Rear_Left_Wheel/>
-    <!-- <xacro:rgb_camera frlr_prefix="front" lrc_prefix="center">
+    <xacro:rgb_camera frlr_prefix="front" lrc_prefix="center">
       <origin xyz="-0.04 0 1" rpy="0 0.087 0"/>
     </xacro:rgb_camera>
     <xacro:VLP-16 parent="chassis" name="velodyne" topic="/velodyne_points" organize_cloud="${organize_cloud}" hz="10" samples="440" gpu="${gpu}">
-      <origin xyz="0 0 0.4" rpy="0 0 0" />
-    </xacro:VLP-16> -->
+      <origin xyz="0 0 0.8" rpy="0 0 0" />
+    </xacro:VLP-16>
       <gazebo>
         <plugin name="p3d" filename="libgazebo_ros_p3d.so">

File: spawn_car/model/urban/urdf/wheels/urban_suspension.urdf.xacro (robot description, xacro)
@@ -46,6 +46,6 @@
             <parent link="chassis"/>
             <child link="fl_axle"/>
-            <origin rpy="${degree_90} 0 0" xyz="${wheel_base/2} ${-front_track/2} 0"/>
-            <axis xyz="0 1 0"/>
+            <origin rpy="${degree_90} 0 0" xyz="${wheel_base/2} ${front_track/2} 0"/>
+            <axis xyz="0 -1 0"/>
             <limit lower="-0.785398" upper="0.785398" effort="500000" velocity="250"/>
         </joint>
@@ -63,6 +63,6 @@
             <parent link="chassis"/>
             <child link="fr_axle"/>
-            <origin rpy="${degree_90} 0 0" xyz="${wheel_base/2} ${front_track/2} 0"/>
-            <axis xyz="0 1 0"/>
+            <origin rpy="${degree_90} 0 0" xyz="${wheel_base/2} ${-front_track/2} 0"/>
+            <axis xyz="0 -1 0"/>
             <limit lower="-0.785398" upper="0.785398" effort="500000" velocity="250"/>
         </joint>
@@ -80,5 +80,5 @@
             <parent link="chassis"/>
             <child link="rear_left_wheel"/>
-            <origin rpy="${degree_90} 0 0" xyz="${-wheel_base/2} ${-front_track/2} 0"/>
+            <origin rpy="${degree_90} 0 0" xyz="${-wheel_base/2} ${front_track/2} 0"/>
             <axis xyz="0 0 -1"/>
             <limit effort="1000" velocity="1000"/>
@@ -90,5 +90,5 @@
             <parent link="chassis"/>
             <child link="rear_right_wheel"/>
-            <origin rpy="${degree_90} 0 0" xyz="${-wheel_base/2} ${front_track/2} 0"/>
+            <origin rpy="${degree_90} 0 0" xyz="${-wheel_base/2} ${-front_track/2} 0"/>
             <axis xyz="0 0 -1"/>
             <limit effort="1000" velocity="1000"/>
