Commit message: Add realsense_gazebo_plugin as a submodule

File: spawn_car/model/urban/urdf/sensors/camera.urdf.xacro (robot description, xacro)
@@ -2,4 +2,7 @@
 <robot xmlns:xacro="http://www.ros.org/wiki/xacro" name="rgb_camera">
   <xacro:macro name="rgb_camera" params="frlr_prefix lrc_prefix *origin">
+    <material name="red">
+      <color rgba="0.8 0.0 0.0 1.0"/>
+    </material>
     <joint name="${frlr_prefix}_${lrc_prefix}_camera_joint" type="fixed">
       <axis xyz="0 1 0" />

File: spawn_car/model/urban/urdf/urban_description.urdf.xacro (robot description, xacro)
@@ -13,4 +13,5 @@
     <xacro:include filename="$(find spawn_car)/model/urban/urdf/sensors/camera.urdf.xacro"/>
     <xacro:include filename="$(find spawn_car)/model/urban/urdf/sensors/vlp-16.urdf.xacro"/>
+    <xacro:include filename="$(find spawn_car)/model/urban/urdf/sensors/_d435.urdf.xacro"/>
     <!-- *************** -->
     <!-- Robots Elements -->
@@ -27,4 +28,10 @@
       <origin xyz="0 0 0.8" rpy="0 0 0" />
     </xacro:VLP-16>
+    <xacro:sensor_d435 parent="chassis" name="camera1">
+      <origin xyz="0.1 0 2.0" rpy="0 0 0"/>
+    </xacro:sensor_d435>
+    <xacro:sensor_d435 parent="chassis" name="camera2">
+      <origin xyz="-0.1 0 2.0" rpy="0 0 3.1456"/>
+    </xacro:sensor_d435>
       <gazebo>
         <plugin name="p3d" filename="libgazebo_ros_p3d.so">
