Commit message: get to code again

File: spawn_car/model/urban/urdf/sensors/_d435.urdf.xacro (robot description, xacro)
@@ -8,5 +8,5 @@
 <robot name="sensor_d435" xmlns:xacro="http://ros.org/wiki/xacro">
   <!--File includes-->
-  <xacro:include filename="$(find realsense2_description)/urdf/_d435.gazebo.xacro"/>
+  <xacro:include filename="$(find spawn_car)/model/urban/urdf/sensors/_d435.gazebo.xacro"/>
   <xacro:macro name="sensor_d435" params="name:=camera topics_ns:=camera parent *origin publish_pointcloud:=true">
     <xacro:property name="M_PI" value="3.1415926535897931" />
@@ -48,6 +48,6 @@
         <geometry>
           <!-- <box size="${d435_cam_width} ${d435_cam_height} ${d435_cam_depth}"/> -->
-          <mesh filename="package://realsense2_description/meshes/d435.dae" />
-          <!-- <mesh filename="package://spawn_car/model/formula/meshes/VLP16_base_2.dae" /> -->
+          <!-- <mesh filename="package://realsense2_description/meshes/d435.dae" /> -->
+          <mesh filename="package://spawn_car/model/urban/meshes/d435.dae"/>
           <!--<mesh filename="package://realsense2_description/meshes/d435/d435.dae" />-->
         </geometry>

File: spawn_car/model/urban/urdf/sensors/camera.urdf.xacro (robot description, xacro)
@@ -20,9 +20,8 @@
       </collision>
       <visual>
-        <origin xyz="0 0 0" rpy="0 0 0"/>
+        <origin xyz="0 0 0" rpy="${degree_90} 0 ${degree_90}"/>
         <geometry>
-          <box size="0.026 0.026 0.0203"/>
+            <mesh filename="package://spawn_car/model/urban/meshes/c270.stl" scale="0.0001 0.0001 0.0001"/>
         </geometry>
-        <material name="red"/>
       </visual>
       <inertial>
@@ -41,5 +40,5 @@
             <mu1>0.2</mu1>
             <mu2>0.2</mu2>
-            <material>Gazebo/Red</material>
+            <material>Gazebo/Grey</material>
             <sensor type="camera" name="${frlr_prefix}_${lrc_prefix}_camera">
                 <update_rate>30.0</update_rate>

File: spawn_car/model/urban/urdf/urban_description.urdf.xacro (robot description, xacro)
@@ -23,14 +23,11 @@
     <xacro:Rear_Left_Wheel/>
     <xacro:rgb_camera frlr_prefix="front" lrc_prefix="center">
-      <origin xyz="-0.04 0 1" rpy="0 0.087 0"/>
+      <origin xyz="0.00 0 0.9" rpy="0 0.087 0"/>
     </xacro:rgb_camera>
     <xacro:VLP-16 parent="chassis" name="velodyne" topic="/velodyne_points" organize_cloud="${organize_cloud}" hz="10" samples="440" gpu="${gpu}">
       <origin xyz="0 0 0.8" rpy="0 0 0" />
     </xacro:VLP-16>
-    <xacro:sensor_d435 parent="chassis" name="camera1">
-      <origin xyz="0.1 0 2.0" rpy="0 0 0"/>
-    </xacro:sensor_d435>
-    <xacro:sensor_d435 parent="chassis" name="camera2">
-      <origin xyz="-0.1 0 2.0" rpy="0 0 3.1456"/>
+    <xacro:sensor_d435 name="camera" topics_ns="camera" parent="chassis" publish_pointcloud="true">
+      <origin xyz="0.6 0 0.4" rpy="0 0 0" />
     </xacro:sensor_d435>
       <gazebo>

File: spawn_car/model/urban/urdf/vehicle_properties.urdf.xacro (robot description, xacro)
@@ -10,4 +10,6 @@
     <xacro:property name = "degree_90" value="1.57079633"/>
     <xacro:property name = "degree_180" value="3.14159265"/>
+    <xacro:property name = "degree_270" value="4.71239"/>
+    <xacro:property name = "degree_360" value="6.28319"/>
     <xacro:property name="car_length" value="1.490" />
     <xacro:property name="car_width" value="0.830" />
