Commit message: fixed package.xml

File: spawn_car/model/urban/urdf/bases/urban_body.urdf.xacro (robot description, xacro)
@@ -39,5 +39,9 @@
                   <mesh filename="file://$(find spawn_car)/model/urban/meshes/SDTwizy.stl" scale="0.008 0.0055 0.0062"/>
                 </geometry>
-              </visual>
+                <material name="chassis_mat">
+                    <color rgba="0.2 0.2 0.2 1"/>
+                    <!-- grey -->
+                </material>
+            </visual>
             <collision>
                 <origin xyz="0.015 0.0 0.015" rpy="0 0 1.57079632679"/>
@@ -45,4 +49,8 @@
                   <mesh filename="file://$(find spawn_car)/model/urban/meshes/SDTwizy_collision.stl" scale="0.008 0.0055 0.0062"/>
                 </geometry>
+                <material name="chassis_mat">
+                    <color rgba="0.2 0.2 0.2 1"/>
+                    <!-- grey -->
+                </material>
             </collision>
             <xacro:inertia_of_body/>

Commit message: get to code again

File: spawn_car/model/urban/urdf/bases/urban_body.urdf.xacro (robot description, xacro)
@@ -14,5 +14,5 @@
         <link name="dummy">
             <visual>
-                <origin xyz="0 0 0" rpy="0 0 0"/>
+                <origin xyz="0 0 0.5" rpy="0 0 0"/>
                 <geometry>
                     <box size="0.001 0.001 0.001"/>
@@ -23,5 +23,5 @@
             <parent link="dummy"/>
             <child link="chassis"/>
-            <origin xyz="0.0 0.0 ${ground_clearance + (chassis_thickness/2)}"/>
+            <origin xyz="0.0 0.0 0.0"/>
             <axis xyz = "0 0 1"/>
         </joint>
@@ -35,7 +35,7 @@
             </visual> -->
             <visual>
-                <origin xyz="0.015 0.0 0.015" rpy="0 0 1.57079632679"/>
+                <origin xyz="0.0 0.0 0.0" rpy="1.57079632679 0 1.57079632679"/>
                 <geometry>
-                  <mesh filename="file://$(find spawn_car)/model/urban/meshes/SDTwizy.stl" scale="0.008 0.0055 0.0062"/>
+                  <mesh filename="file://$(find spawn_car)/model/urban/meshes/Car_body_transformed.stl" scale="0.001 0.001 0.001"/>
                 </geometry>
                 <material name="chassis_mat">
@@ -45,7 +45,7 @@
             </visual>
             <collision>
-                <origin xyz="0.015 0.0 0.015" rpy="0 0 1.57079632679"/>
+                <origin xyz="0.0 0.0 0.0" rpy="1.57079632679 0 1.57079632679"/>
                 <geometry>
-                  <mesh filename="file://$(find spawn_car)/model/urban/meshes/SDTwizy_collision.stl" scale="0.008 0.0055 0.0062"/>
+                  <mesh filename="file://$(find spawn_car)/model/urban/meshes/Car_body_transformed.stl" scale="0.001 0.001 0.001"/>
                 </geometry>
                 <material name="chassis_mat">

File: spawn_car/model/urban/urdf/sensors/_d435.gazebo.xacro (robot description, xacro)
@@ -43,5 +43,5 @@
         <always_on>1</always_on>
         <update_rate>30</update_rate>
-        <visualize>1</visualize>
+        <visualize>0</visualize>
       </sensor>
       <sensor name="${camera_name}ired1" type="camera">

File: spawn_car/model/urban/urdf/urban_description.urdf.xacro (robot description, xacro)
@@ -22,12 +22,12 @@
     <xacro:Rear_Right_Wheel/>
     <xacro:Rear_Left_Wheel/>
-    <xacro:rgb_camera frlr_prefix="front" lrc_prefix="center">
-      <origin xyz="0.00 0 0.9" rpy="0 0.087 0"/>
-    </xacro:rgb_camera>
+    <!-- <xacro:rgb_camera frlr_prefix="front" lrc_prefix="center">
+      <origin xyz="0.3 0 1.39" rpy="0 0.087 0"/>
+    </xacro:rgb_camera> -->
     <xacro:VLP-16 parent="chassis" name="velodyne" topic="/velodyne_points" organize_cloud="${organize_cloud}" hz="10" samples="440" gpu="${gpu}">
-      <origin xyz="0 0 0.8" rpy="0 0 0" />
+      <origin xyz="0.3 0 1.30" rpy="0 0 0" />
     </xacro:VLP-16>
     <xacro:sensor_d435 name="camera" topics_ns="camera" parent="chassis" publish_pointcloud="true">
-      <origin xyz="0.6 0 0.4" rpy="0 0 0" />
+      <origin xyz="0.8 0 0.4" rpy="0 0 0" />
     </xacro:sensor_d435>
       <gazebo>

File: spawn_car/model/urban/urdf/vehicle_properties.urdf.xacro (robot description, xacro)
@@ -24,6 +24,6 @@
     <xacro:property name="chassis_width" value="0.830" />
     <xacro:property name="chassis_length" value="1.49" />
-    <xacro:property name="chassis_thickness" value="0.03" />
-    <xacro:property name="chassis_mass" value="200" />
+    <xacro:property name="chassis_thickness" value="1.00" />
+    <xacro:property name="chassis_mass" value="250" />
        <!-- variable -->
     <!-- aluminium density is 2.7 g/cm³ or 2700 kg/m3-->
@@ -35,8 +35,8 @@
     -->
     <xacro:property name="wheel_cylindrical_transform" value="1.570795" />
-    <xacro:property name="front_tyre_radius" value="0.172"/>
+    <xacro:property name="front_tyre_radius" value="0.19"/>
     <xacro:property name="front_tyre_width" value="0.125"/>
     <xacro:property name="front_tyre_mass" value="10.0"/>
-    <xacro:property name="rear_tyre_radius" value="0.172"/>
+    <xacro:property name="rear_tyre_radius" value="0.19"/>
     <xacro:property name="rear_tyre_width" value="0.125"/>
     <xacro:property name="rear_tyre_mass" value="10.0"/>

File: spawn_car/model/urban/urdf/wheels/urban_suspension.urdf.xacro (robot description, xacro)
@@ -6,5 +6,6 @@
 <robot xmlns:xacro="http://www.ros.org/wiki/xacro" name="suspension urdf">
     <material name="tire_mat">
-        <color rgba="1 1 1 1"/>
+        <!-- <color rgba="1 1 1 1"/> -->
+        <color rgba="0.35 0.35 0.35 1.0" />
     </material>
     <xacro:include filename="$(find spawn_car)/model/urban/urdf/wheels/suspension.gazebo.xacro"/>
@@ -46,5 +47,5 @@
             <parent link="chassis"/>
             <child link="fl_axle"/>
-            <origin rpy="${degree_90} 0 0" xyz="${wheel_base/2} ${front_track/2} 0"/>
+            <origin rpy="${degree_90} 0 0" xyz="${wheel_base/2} ${front_track/2} ${front_tyre_radius - ground_clearance}"/>
             <axis xyz="0 -1 0"/>
             <limit lower="-0.785398" upper="0.785398" effort="500000" velocity="250"/>
@@ -63,5 +64,5 @@
             <parent link="chassis"/>
             <child link="fr_axle"/>
-            <origin rpy="${degree_90} 0 0" xyz="${wheel_base/2} ${-front_track/2} 0"/>
+            <origin rpy="${degree_90} 0 0" xyz="${wheel_base/2} ${-front_track/2} ${front_tyre_radius - ground_clearance}"/>
             <axis xyz="0 -1 0"/>
             <limit lower="-0.785398" upper="0.785398" effort="500000" velocity="250"/>
@@ -80,5 +81,5 @@
             <parent link="chassis"/>
             <child link="rear_left_wheel"/>
-            <origin rpy="${degree_90} 0 0" xyz="${-wheel_base/2} ${front_track/2} 0"/>
+            <origin rpy="${degree_90} 0 0" xyz="${-wheel_base/2} ${rear_track/2} ${rear_tyre_radius - ground_clearance - 0.02}"/>
             <axis xyz="0 0 -1"/>
             <limit effort="1000" velocity="1000"/>
@@ -90,5 +91,5 @@
             <parent link="chassis"/>
             <child link="rear_right_wheel"/>
-            <origin rpy="${degree_90} 0 0" xyz="${-wheel_base/2} ${-front_track/2} 0"/>
+            <origin rpy="${degree_90} 0 0" xyz="${-wheel_base/2} ${-rear_track/2} ${rear_tyre_radius - ground_clearance - 0.02}"/>
             <axis xyz="0 0 -1"/>
             <limit effort="1000" velocity="1000"/>
@@ -98,16 +99,16 @@
     <link name="fl_axle">
         <inertial>
-          <mass value="1"/>
-          <origin xyz="0 0 0"/>
-          <inertia ixx="0.004" ixy="0.0" ixz="0.0" iyy="0.004" iyz="0.0" izz="0.004"/>
+            <mass value="1"/>
+            <origin xyz="0 0 0"/>
+            <inertia ixx="0.004" ixy="0.0" ixz="0.0" iyy="0.004" iyz="0.0" izz="0.004"/>
         </inertial>
         <collision>
             <geometry>
-              <box size="0.05 0.05 0.15" />
+                <box size="0.005 0.005 0.005" />
             </geometry>
         </collision>
         <visual>
             <geometry>
-              <box size="0.05 0.05 0.15" />
+                <box size="0.005 0.005 0.005" />
             </geometry>
         </visual>
@@ -121,10 +122,10 @@
         <collision>
             <geometry>
-              <box size="0.05 0.05 0.15" />
+              <box size="0.005 0.005 0.005" />
             </geometry>
         </collision>
         <visual>
             <geometry>
-              <box size="0.05 0.05 0.15" />
+              <box size="0.005 0.005 0.005" />
             </geometry>
         </visual>
@@ -134,5 +135,5 @@
             <origin rpy="0 0 0" xyz="0 0 0"/>
             <geometry>
-                <cylinder length="${front_tyre_width}" radius="${front_tyre_radius}"/>
+                <mesh filename="file://$(find spawn_car)/model/urban/meshes/mevi_tire.stl" scale="0.001 0.001 0.001"/>
             </geometry>
             <material name="tire_mat"/>
@@ -141,5 +142,5 @@
             <origin rpy="0 0 0" xyz="0 0 0"/>
             <geometry>
-                <cylinder length="${front_tyre_width}" radius="${front_tyre_radius}"/>
+                <mesh filename="file://$(find spawn_car)/model/urban/meshes/mevi_tire.stl" scale="0.001 0.001 0.001"/>
             </geometry>
         </collision>
@@ -150,5 +151,5 @@
             <origin rpy="0 0 0" xyz="0 0 0"/>
             <geometry>
-                <cylinder length="${front_tyre_width}" radius="${front_tyre_radius}"/>
+                <mesh filename="file://$(find spawn_car)/model/urban/meshes/mevi_tire.stl" scale="0.001 0.001 0.001"/>
             </geometry>
             <material name="tire_mat"/>
@@ -157,5 +158,5 @@
             <origin rpy="0 0 0" xyz="0 0 0"/>
             <geometry>
-                <cylinder length="${front_tyre_width}" radius="${front_tyre_radius}"/>
+                <mesh filename="file://$(find spawn_car)/model/urban/meshes/mevi_tire.stl" scale="0.001 0.001 0.001"/>
             </geometry>
         </collision>

Commit message: add pure pursuit and some junction speed configuration

File: spawn_car/model/urban/urdf/bases/urban_body.urdf.xacro (robot description, xacro)
@@ -14,5 +14,5 @@
         <link name="dummy">
             <visual>
-                <origin xyz="0 0 0.5" rpy="0 0 0"/>
+                <origin xyz="0.0 0.0 0.5" rpy="0 0 0"/>
                 <geometry>
                     <box size="0.001 0.001 0.001"/>

File: spawn_car/model/urban/urdf/urban_description.urdf.xacro (robot description, xacro)
@@ -25,10 +25,10 @@
       <origin xyz="0.3 0 1.39" rpy="0 0.087 0"/>
     </xacro:rgb_camera> -->
-    <xacro:VLP-16 parent="chassis" name="velodyne" topic="/velodyne_points" organize_cloud="${organize_cloud}" hz="10" samples="440" gpu="${gpu}">
+    <!-- <xacro:VLP-16 parent="chassis" name="velodyne" topic="/velodyne_points" organize_cloud="${organize_cloud}" hz="10" samples="440" gpu="${gpu}">
       <origin xyz="0.3 0 1.30" rpy="0 0 0" />
     </xacro:VLP-16>
     <xacro:sensor_d435 name="camera" topics_ns="camera" parent="chassis" publish_pointcloud="true">
       <origin xyz="0.8 0 0.4" rpy="0 0 0" />
-    </xacro:sensor_d435>
+    </xacro:sensor_d435>   -->
       <gazebo>
         <plugin name="p3d" filename="libgazebo_ros_p3d.so">
@@ -73,5 +73,5 @@
         </actuator>
           <joint name="rear_left_wheel_joint">
-            <hardwareInterface>hardware_interface/VelocityJointInterface</hardwareInterface>
+            <hardwareInterface>hardware_interface/EffortJointInterface</hardwareInterface>
           </joint>
       </transmission>
@@ -82,5 +82,5 @@
         </actuator>
           <joint name="rear_right_wheel_joint">
-            <hardwareInterface>hardware_interface/VelocityJointInterface</hardwareInterface>
+            <hardwareInterface>hardware_interface/EffortJointInterface</hardwareInterface>
           </joint>
       </transmission>
